Commit message: got the robot_state_publisher working, and a super simple URDF loaded into rviz2

File: turtle_brick/urdf/turtle.urdf.xacro (robot description, xacro)
@@ -7,4 +7,5 @@
         <child link="base_link"/>
     </joint>
+    <link name="base_link">
         <visual>
             <origin xyz="0 0 0.05" rpy="0 0 0"/>

Commit message: got the joint_state_publisher and GUI to work, as well as the base_link movemtn in rviz

File: turtle_brick/urdf/turtle.urdf.xacro (robot description, xacro)
@@ -1,15 +1,42 @@
 <?xml version="1.0"?>
 <robot xmlns:xacro="http://www.ros.org/wiki/xacro" name="turtle">
+    <!-- WIP NEED TO ENABLE PARAMETERS FOR THIS URDF -->
     <link name="world"></link>
+    <!-- odom is the fixed starting position of the turtle robot -->
+    <joint name="odom_joint" type="fixed">
+        <origin xyz="3 3 0" rpy="0 0 0"/>
+        <parent link="world"/>
+        <child link="odom"/>
+    </joint>
+    <link name="odom"></link>
+    <!-- the turtle robot can move anywhere along the xy plane -->
+    <!-- floating and planar joint types do not work so implement a cartesian workaround -->
+    <joint name="x_joint" type="prismatic">
+        <origin xyz="0 0 0" rpy="0 0 0"/>
+        <parent link="odom"/>
+        <child link="x_link"/>
+        <limit lower="-5" upper="5" velocity="100" effort="100"/>
+        <axis xyz="1 0 0"/>
+    </joint>
+    <link name="x_link"></link>
+    <joint name="y_joint" type="prismatic">
+        <origin xyz="0 0 0" rpy="0 0 0"/>
+        <parent link="x_link"/>
+        <child link="y_link"/>
+        <limit lower="-5" upper="5" velocity="100" effort="100"/>
+        <axis xyz="0 1 0"/>
+    </joint>
+    <link name="y_link"></link>
+    <!-- the turtle robot base_link -->
     <joint name="base_joint" type="fixed">
-        <origin xyz="1.5 1.0 0" rpy="0 0 0"/>
-        <parent link="world"/>
+        <origin xyz="0 0 0" rpy="0 0 0"/>
+        <parent link="y_link"/>
         <child link="base_link"/>
     </joint>
     <link name="base_link">
         <visual>
-            <origin xyz="0 0 0.05" rpy="0 0 0"/>
+            <origin xyz="0 0 0" rpy="0 0 0"/>
             <geometry>
-                <box size="2.5 1.5 0.1" />
+                <box size="0.5 0.5 0.5" />
             </geometry>
             <material name="green">
@@ -18,14 +45,32 @@
         </visual>
         <collision>
-            <origin xyz="0 0 0.05" rpy="0 0 0"/>
+            <origin xyz="0 0 0" rpy="0 0 0"/>
             <geometry>
-                <box size="2.5 1.5 0.1" />
+                <box size="0.5 0.5 0.5" />
             </geometry>
         </collision>
-        <inertial>
-            <origin xyz="0 0 0.05" rpy="0 0 0"/>
-            <mass value="12" />
-            <inertia ixx="2.26" ixy="0.0" ixz="0.0" iyy="6.26" iyz="0.0" izz="8.5" />
-        </inertial>
     </link>
+<!--
+    <joint name="cylindrical_joint" type="fixed">
+        <origin xyz="0 0 0" rpy="0 0 0"/>
+        <parent link="y_link"/>
+        <child link="base_link"/>
+    </joint>
+    <link name="cylindrical_link">
+        <visual>
+            <origin xyz="0 0 0" rpy="0 0 0"/>
+            <geometry>
+                <box size="0.5 0.5 0.5" />
+            </geometry>
+            <material name="green">
+                <color rgba="0.2 1 0.2 1"/>
+            </material>
+        </visual>
+        <collision>
+            <origin xyz="0 0 0" rpy="0 0 0"/>
+            <geometry>
+                <box size="0.5 0.5 0.5" />
+            </geometry>
+        </collision>
+    </link> -->
 </robot>

Commit message: completely wrong approach regarding the movement and translation, there is no world and odom links, only frames/tfs

File: turtle_brick/urdf/turtle.urdf.xacro (robot description, xacro)
@@ -5,9 +5,10 @@
     <!-- odom is the fixed starting position of the turtle robot -->
     <joint name="odom_joint" type="fixed">
-        <origin xyz="3 3 0" rpy="0 0 0"/>
+        <origin xyz="1 1 0" rpy="0 0 0"/>
         <parent link="world"/>
         <child link="odom"/>
     </joint>
     <link name="odom"></link>
+    <!-- movement and rotation of the turtle 'unicycle' -->
     <!-- the turtle robot can move anywhere along the xy plane -->
     <!-- floating and planar joint types do not work so implement a cartesian workaround -->
@@ -16,5 +17,5 @@
         <parent link="odom"/>
         <child link="x_link"/>
-        <limit lower="-5" upper="5" velocity="100" effort="100"/>
+        <limit lower="-5" upper="5" velocity="100" effort="1000.0"/>
         <axis xyz="1 0 0"/>
     </joint>
@@ -24,5 +25,5 @@
         <parent link="x_link"/>
         <child link="y_link"/>
-        <limit lower="-5" upper="5" velocity="100" effort="100"/>
+        <limit lower="-5" upper="5" velocity="100" effort="1000.0"/>
         <axis xyz="0 1 0"/>
     </joint>
@@ -30,11 +31,11 @@
     <!-- the turtle robot base_link -->
     <joint name="base_joint" type="fixed">
-        <origin xyz="0 0 0" rpy="0 0 0"/>
-        <parent link="y_link"/>
+        <origin xyz="0 0 1" rpy="0 0 0"/>
+        <parent link="stem_link"/>
         <child link="base_link"/>
     </joint>
     <link name="base_link">
         <visual>
-            <origin xyz="0 0 0" rpy="0 0 0"/>
+            <origin xyz="0 0 0.25" rpy="0 0 0"/>
             <geometry>
                 <box size="0.5 0.5 0.5" />
@@ -51,26 +52,91 @@
         </collision>
     </link>
-<!--
-    <joint name="cylindrical_joint" type="fixed">
+    <!-- the turtle robot can turn around on its wheel -->
+    <joint name="rotate_joint" type="continuous">
         <origin xyz="0 0 0" rpy="0 0 0"/>
         <parent link="y_link"/>
-        <child link="base_link"/>
+        <child link="rotate_link"/>
+        <axis xyz="0 0 1"/>
+        <limit effort="1000.0" velocity="0.5"/>
     </joint>
-    <link name="cylindrical_link">
+    <link name="rotate_link"></link>
+    <!-- bottom half of the turtle 'unicycle' -->
+    <!-- WIP need to change wheel origin for parameters -->
+    <joint name="wheel_joint" type="continuous">
+        <origin xyz="0 0 0.25" rpy="1.57079632679 0 0"/>
+        <parent link="rotate_link"/>
+        <child link="wheel_link"/>
+        <axis xyz="0 1 0"/>
+        <limit effort="1000.0" velocity="0.5"/>
+    </joint>
+    <!-- WIP need to change wheel radius for parameters -->
+    <link name="wheel_link">
         <visual>
             <origin xyz="0 0 0" rpy="0 0 0"/>
             <geometry>
-                <box size="0.5 0.5 0.5" />
+                <cylinder length="0.05" radius="0.25"/>
             </geometry>
-            <material name="green">
-                <color rgba="0.2 1 0.2 1"/>
+            <material name="red">
+                <color rgba="1 0.2 0.2 1"/>
+            </material>
+        </visual>
+    </link>
+    <joint name="stem_joint" type="fixed">
+        <origin xyz="0 0 0.25" rpy="1.57079632679 0 0"/>
+        <parent link="wheel_link"/>
+        <child link="stem_link"/>
+    </joint>
+    <link name="stem_link">
+        <visual>
+            <origin xyz="0 0 0.5" rpy="0 0 0"/>
+            <geometry>
+                <cylinder length="1" radius="0.05"/>
+            </geometry>
+            <material name="red">
+                <color rgba="1 0.2 0.2 1"/>
+            </material>
+        </visual>
+    </link>
+    <!-- top half of the turtle 'unicycle' -->
+    <joint name="cylindrical_joint" type="fixed">
+        <origin xyz="0 0 0.25" rpy="0 0 0"/>
+        <parent link="base_link"/>
+        <child link="cylindrical_link"/>
+    </joint>
+    <!-- WIP need to change height for parameters -->
+    <link name="cylindrical_link">
+        <visual>
+            <origin xyz="0 0 0.5" rpy="0 0 0"/>
+            <geometry>
+                <cylinder length="1" radius="0.05"/>
+            </geometry>
+            <material name="red">
+                <color rgba="1 0.2 0.2 1"/>
+            </material>
+        </visual>
+    </link>
+    <joint name="platform_joint" type="revolute">
+        <origin xyz="0 0 1" rpy="0 0 0"/>
+        <parent link="cylindrical_link"/>
+        <child link="platform_link"/>
+        <axis xyz="0 1 0"/>
+        <limit effort="1000.0" lower="-0.5" upper="0.5" velocity="0.5"/>
+    </joint>
+    <link name="platform_link">
+        <visual>
+            <origin xyz="0 0 -0.005" rpy="0 0 0"/>
+            <geometry>
+                <cylinder length="0.01" radius="0.5"/>
+            </geometry>
+            <material name="blue">
+                <color rgba="0.2 0.2 1 1"/>
             </material>
         </visual>
         <collision>
-            <origin xyz="0 0 0" rpy="0 0 0"/>
+            <origin xyz="0 0 -0.005" rpy="0 0 0"/>
             <geometry>
-                <box size="0.5 0.5 0.5" />
+                <cylinder length="0.01" radius="0.5"/>
             </geometry>
         </collision>
-    </link> -->
+    </link>
 </robot>

Commit message: finished 90% of the urdf stuff, just need to implement .yaml files

File: turtle_brick/urdf/turtle.urdf.xacro (robot description, xacro)
@@ -1,43 +1,23 @@
 <?xml version="1.0"?>
 <robot xmlns:xacro="http://www.ros.org/wiki/xacro" name="turtle">
-    <!-- WIP NEED TO ENABLE PARAMETERS FOR THIS URDF -->
-    <link name="world"></link>
-    <!-- odom is the fixed starting position of the turtle robot -->
-    <joint name="odom_joint" type="fixed">
-        <origin xyz="1 1 0" rpy="0 0 0"/>
-        <parent link="world"/>
-        <child link="odom"/>
-    </joint>
-    <link name="odom"></link>
-    <!-- movement and rotation of the turtle 'unicycle' -->
-    <!-- the turtle robot can move anywhere along the xy plane -->
-    <!-- floating and planar joint types do not work so implement a cartesian workaround -->
-    <joint name="x_joint" type="prismatic">
-        <origin xyz="0 0 0" rpy="0 0 0"/>
-        <parent link="odom"/>
-        <child link="x_link"/>
-        <limit lower="-5" upper="5" velocity="100" effort="1000.0"/>
-        <axis xyz="1 0 0"/>
-    </joint>
-    <link name="x_link"></link>
-    <joint name="y_joint" type="prismatic">
-        <origin xyz="0 0 0" rpy="0 0 0"/>
-        <parent link="x_link"/>
-        <child link="y_link"/>
-        <limit lower="-5" upper="5" velocity="100" effort="1000.0"/>
-        <axis xyz="0 1 0"/>
-    </joint>
-    <link name="y_link"></link>
+    <!-- platform_height is the same as total height of the turtle -->
+    <xacro:property name="platform_height" value="3"/>
+    <xacro:property name="wheel_radius" value="0.5"/>
+    <!-- constant dimensions -->
+    <xacro:property name="base_length" value="0.125"/>
+    <xacro:property name="cylinder_radius" value="${base_length/2}"/>
+    <xacro:property name="stem_radius" value="${base_length/2}"/>
+    <xacro:property name="platform_radius" value="0.5"/>
+    <xacro:property name="platform_thickness" value="0.05"/>
+    <xacro:property name="wheel_thickness" value="0.1"/>
+    <!-- dimensions adaptive to parameters -->
+    <xacro:property name="stem_height" value="${wheel_radius}"/>
+    <xacro:property name="cylinder_height" value="${platform_height - (wheel_radius + stem_height + base_length + platform_thickness)}"/>
     <!-- the turtle robot base_link -->
-    <joint name="base_joint" type="fixed">
-        <origin xyz="0 0 1" rpy="0 0 0"/>
-        <parent link="stem_link"/>
-        <child link="base_link"/>
-    </joint>
     <link name="base_link">
         <visual>
-            <origin xyz="0 0 0.25" rpy="0 0 0"/>
+            <origin xyz="0 0 ${base_length/2}" rpy="0 0 0"/>
             <geometry>
-                <box size="0.5 0.5 0.5" />
+                <box size="${base_length} ${base_length} ${base_length}" />
             </geometry>
             <material name="green">
@@ -45,69 +25,16 @@
             </material>
         </visual>
-        <collision>
-            <origin xyz="0 0 0" rpy="0 0 0"/>
-            <geometry>
-                <box size="0.5 0.5 0.5" />
-            </geometry>
-        </collision>
-    </link>
-    <!-- the turtle robot can turn around on its wheel -->
-    <joint name="rotate_joint" type="continuous">
-        <origin xyz="0 0 0" rpy="0 0 0"/>
-        <parent link="y_link"/>
-        <child link="rotate_link"/>
-        <axis xyz="0 0 1"/>
-        <limit effort="1000.0" velocity="0.5"/>
-    </joint>
-    <link name="rotate_link"></link>
-    <!-- bottom half of the turtle 'unicycle' -->
-    <!-- WIP need to change wheel origin for parameters -->
-    <joint name="wheel_joint" type="continuous">
-        <origin xyz="0 0 0.25" rpy="1.57079632679 0 0"/>
-        <parent link="rotate_link"/>
-        <child link="wheel_link"/>
-        <axis xyz="0 1 0"/>
-        <limit effort="1000.0" velocity="0.5"/>
-    </joint>
-    <!-- WIP need to change wheel radius for parameters -->
-    <link name="wheel_link">
-        <visual>
-            <origin xyz="0 0 0" rpy="0 0 0"/>
-            <geometry>
-                <cylinder length="0.05" radius="0.25"/>
-            </geometry>
-            <material name="red">
-                <color rgba="1 0.2 0.2 1"/>
-            </material>
-        </visual>
-    </link>
-    <joint name="stem_joint" type="fixed">
-        <origin xyz="0 0 0.25" rpy="1.57079632679 0 0"/>
-        <parent link="wheel_link"/>
-        <child link="stem_link"/>
-    </joint>
-    <link name="stem_link">
-        <visual>
-            <origin xyz="0 0 0.5" rpy="0 0 0"/>
-            <geometry>
-                <cylinder length="1" radius="0.05"/>
-            </geometry>
-            <material name="red">
-                <color rgba="1 0.2 0.2 1"/>
-            </material>
-        </visual>
     </link>
     <!-- top half of the turtle 'unicycle' -->
-    <joint name="cylindrical_joint" type="fixed">
-        <origin xyz="0 0 0.25" rpy="0 0 0"/>
+    <joint name="cylinder_joint" type="fixed">
+        <origin xyz="0 0 ${base_length}" rpy="0 0 0"/>
         <parent link="base_link"/>
-        <child link="cylindrical_link"/>
+        <child link="cylinder_link"/>
     </joint>
-    <!-- WIP need to change height for parameters -->
-    <link name="cylindrical_link">
+    <link name="cylinder_link">
         <visual>
-            <origin xyz="0 0 0.5" rpy="0 0 0"/>
+            <origin xyz="0 0 ${cylinder_height/2}" rpy="0 0 0"/>
             <geometry>
-                <cylinder length="1" radius="0.05"/>
+                <cylinder length="${cylinder_height}" radius="${cylinder_radius}"/>
             </geometry>
             <material name="red">
@@ -117,6 +44,6 @@
     </link>
     <joint name="platform_joint" type="revolute">
-        <origin xyz="0 0 1" rpy="0 0 0"/>
-        <parent link="cylindrical_link"/>
+        <origin xyz="0 0 ${cylinder_height}" rpy="0 0 0"/>
+        <parent link="cylinder_link"/>
         <child link="platform_link"/>
         <axis xyz="0 1 0"/>
@@ -125,7 +52,7 @@
     <link name="platform_link">
         <visual>
-            <origin xyz="0 0 -0.005" rpy="0 0 0"/>
+            <origin xyz="0 0 ${platform_thickness/2}" rpy="0 0 0"/>
             <geometry>
-                <cylinder length="0.01" radius="0.5"/>
+                <cylinder length="${platform_thickness}" radius="${platform_radius}"/>
             </geometry>
             <material name="blue">
@@ -134,9 +61,45 @@
         </visual>
         <collision>
-            <origin xyz="0 0 -0.005" rpy="0 0 0"/>
+            <origin xyz="0 0 ${platform_thickness/2}" rpy="0 0 0"/>
             <geometry>
-                <cylinder length="0.01" radius="0.5"/>
+                <cylinder length="${platform_thickness}" radius="${platform_radius}"/>
             </geometry>
         </collision>
     </link>
+    <!-- bottom half of the turtle 'unicycle' -->
+    <joint name="stem_joint" type="continuous">
+        <origin xyz="0 0 0" rpy="0 0 0"/>
+        <parent link="base_link"/>
+        <child link="stem_link"/>
+        <axis xyz="0 0 1"/>
+    </joint>
+    <link name="stem_link">
+        <visual>
+            <origin xyz="0 0 -${stem_height/2}" rpy="0 0 0"/>
+            <geometry>
+                <cylinder length="${stem_height}" radius="${stem_radius}"/>
+            </geometry>
+            <material name="red">
+                <color rgba="1 0.2 0.2 1"/>
+            </material>
+        </visual>
+    </link>
+    <joint name="wheel_joint" type="continuous">
+        <origin xyz="0 0 -${wheel_radius}" rpy="1.57079632679 0 0"/>
+        <parent link="stem_link"/>
+        <child link="wheel_link"/>
+        <axis xyz="0 0 1"/>
+        <limit effort="1000.0" velocity="0.5"/>
+    </joint>
+    <link name="wheel_link">
+        <visual>
+            <origin xyz="0 0 0" rpy="0 0 0"/>
+            <geometry>
+                <cylinder length="${wheel_thickness}" radius="${wheel_radius}"/>
+            </geometry>
+            <material name="red">
+                <color rgba="1 0.2 0.2 1"/>
+            </material>
+        </visual>
+    </link>
 </robot>

Commit message: touched up launch file to include rviz, but still can't figure out how to combine the yaml and xacro files together

File: turtle_brick/urdf/turtle.urdf.xacro (robot description, xacro)
@@ -1,7 +1,9 @@
 <?xml version="1.0"?>
 <robot xmlns:xacro="http://www.ros.org/wiki/xacro" name="turtle">
+    <!-- <xacro:property name="yaml_file" value="$(find turtle_brick)/config/turtle.yaml" />
+    <xacro:property name="props" value="${xacro.load_yaml(yaml_file)}" /> -->
     <!-- platform_height is the same as total height of the turtle -->
-    <xacro:property name="platform_height" value="3"/>
-    <xacro:property name="wheel_radius" value="0.5"/>
+    <xacro:property name="platform_height" value="2"/>
+    <xacro:property name="wheel_radius" value="0.2"/>
     <!-- constant dimensions -->
     <xacro:property name="base_length" value="0.125"/>

Commit message: implemented yaml with xacro and turtle_robot node

File: turtle_brick/urdf/turtle.urdf.xacro (robot description, xacro)
@@ -1,9 +1,10 @@
 <?xml version="1.0"?>
 <robot xmlns:xacro="http://www.ros.org/wiki/xacro" name="turtle">
-    <!-- <xacro:property name="yaml_file" value="$(find turtle_brick)/config/turtle.yaml" />
-    <xacro:property name="props" value="${xacro.load_yaml(yaml_file)}" /> -->
+    <!-- loading in parameter file -->
+    <xacro:property name="yaml_file" value="$(find turtle_brick)/config/turtle.yaml" />
+    <xacro:property name="props" value="${xacro.load_yaml(yaml_file)['/**']['ros__parameters']}" />
     <!-- platform_height is the same as total height of the turtle -->
-    <xacro:property name="platform_height" value="2"/>
-    <xacro:property name="wheel_radius" value="0.2"/>
+    <xacro:property name="platform_height" value="${props['platform_height']}"/>
+    <xacro:property name="wheel_radius" value="${props['wheel_radius']}"/>
     <!-- constant dimensions -->
     <xacro:property name="base_length" value="0.125"/>

Commit message: tried to get tf listener working for robot posiiton, but won't work; will use turtlesim pose instead for now

File: turtle_brick/urdf/turtle.urdf.xacro (robot description, xacro)
@@ -7,9 +7,9 @@
     <xacro:property name="platform_height" value="${props['platform_height']}"/>
     <xacro:property name="wheel_radius" value="${props['wheel_radius']}"/>
+    <xacro:property name="platform_radius" value="${props['platform_radius']}"/>
     <!-- constant dimensions -->
     <xacro:property name="base_length" value="0.125"/>
     <xacro:property name="cylinder_radius" value="${base_length/2}"/>
     <xacro:property name="stem_radius" value="${base_length/2}"/>
-    <xacro:property name="platform_radius" value="0.5"/>
     <xacro:property name="platform_thickness" value="0.05"/>
     <xacro:property name="wheel_thickness" value="0.1"/>

Commit message: made each link a diff color as instructed

File: turtle_brick/urdf/turtle.urdf.xacro (robot description, xacro)
@@ -59,5 +59,5 @@
                 <cylinder length="${platform_thickness}" radius="${platform_radius}"/>
             </geometry>
-            <material name="blue">
+            <material name = "blue">
                 <color rgba="0.2 0.2 1 1"/>
             </material>
@@ -83,6 +83,6 @@
                 <cylinder length="${stem_height}" radius="${stem_radius}"/>
             </geometry>
-            <material name="red">
-                <color rgba="1 0.2 0.2 1"/>
+            <material name="yellow">
+                <color rgba="1 1 0.2 1"/>
             </material>
         </visual>
@@ -101,6 +101,6 @@
                 <cylinder length="${wheel_thickness}" radius="${wheel_radius}"/>
             </geometry>
-            <material name="red">
-                <color rgba="1 0.2 0.2 1"/>
+            <material name="orange">
+                <color rgba="1 0.5 0.1 1"/>
             </material>
         </visual>

Commit message: added collision geometry to URDF

File: turtle_brick/urdf/turtle.urdf.xacro (robot description, xacro)
@@ -28,4 +28,13 @@
             </material>
         </visual>
+        <collision>
+            <origin xyz="0 0 ${base_length/2}" rpy="0 0 0"/>
+            <geometry>
+                <box size="${base_length} ${base_length} ${base_length}" />
+            </geometry>
+            <material name="green">
+                <color rgba="0.2 1 0.2 1"/>
+            </material>
+        </collision>
     </link>
     <!-- top half of the turtle 'unicycle' -->
@@ -45,4 +54,13 @@
             </material>
         </visual>
+        <collision>
+            <origin xyz="0 0 ${cylinder_height/2}" rpy="0 0 0"/>
+            <geometry>
+                <cylinder length="${cylinder_height}" radius="${cylinder_radius}"/>
+            </geometry>
+            <material name="red">
+                <color rgba="1 0.2 0.2 1"/>
+            </material>
+        </collision>
     </link>
     <joint name="platform_joint" type="revolute">
@@ -87,4 +105,13 @@
             </material>
         </visual>
+        <collision>
+            <origin xyz="0 0 -${stem_height/2}" rpy="0 0 0"/>
+            <geometry>
+                <cylinder length="${stem_height}" radius="${stem_radius}"/>
+            </geometry>
+            <material name="yellow">
+                <color rgba="1 1 0.2 1"/>
+            </material>
+        </collision>
     </link>
     <joint name="wheel_joint" type="continuous">
@@ -105,4 +132,13 @@
             </material>
         </visual>
+        <collision>
+            <origin xyz="0 0 0" rpy="0 0 0"/>
+            <geometry>
+                <cylinder length="${wheel_thickness}" radius="${wheel_radius}"/>
+            </geometry>
+            <material name="orange">
+                <color rgba="1 0.5 0.1 1"/>
+            </material>
+        </collision>
     </link>
 </robot>
